Commit message: feat: add rtab with launch files

File: urdf/udacity_bot.xacro (robot description, xacro)
@@ -2,8 +2,8 @@
 <robot name="udacity_bot" xmlns:xacro="http://www.ros.org/wiki/xacro">
   <xacro:include filename="$(find slam_project)/urdf/udacity_bot.gazebo" />
-<link name="robot_footprint"></link>
-  <joint name="robot_footprint_joint" type="fixed">
+<link name="base_footprint"></link>
+  <joint name="base_footprint_joint" type="fixed">
     <origin xyz="0 0 0" rpy="0 0 0" />
-    <parent link="robot_footprint"/>
+    <parent link="base_footprint"/>
     <child link="chassis" />
   </joint>
